File: PCB/NomadKeyboard.kicad_sch (KiCad schematic)
At the start: 94 parts, among them J1 4PIN, J2 OLED, P1 i2c_pin, P2 i2c_pin, SW1 SW_PUSH_LED, SW10 SW_PUSH_LED, SW11 SW_PUSH_LED, SW12 SW_PUSH_LED, SW13 SW_PUSH_LED, SW14 SW_PUSH_LED, SW15 SW_PUSH_LED, SW16 SW_PUSH_LED, SW17 SW_PUSH_LED, SW18 SW_PUSH_LED, SW19 SW_PUSH_LED, SW2 SW_PUSH_LED, SW20 SW_PUSH_LED, SW21 SW_PUSH_LED, SW22 SW_PUSH_LED, SW23 SW_PUSH_LED, SW24 SW_PUSH_LED, SW25 SW_PUSH_LED, SW26 SW_PUSH_LED, SW27 SW_PUSH_LED, SW28 SW_PUSH_LED, SW29 SW_PUSH_LED, SW3 SW_PUSH_LED, SW30 SW_PUSH_LED, SW31 SW_PUSH_LED, SW32 SW_PUSH_LED, SW33 SW_PUSH_LED, SW34 SW_PUSH_LED, SW4 SW_PUSH_LED, SW5 SW_PUSH_LED, SW6 SW_PUSH_LED, SW7 SW_PUSH_LED, SW8 SW_PUSH_LED, SW9 SW_PUSH_LED, U1 ProMicro

Commit message: added new buttons
Parts:
- removed J2: OLED, SofleChoc:OLED_4Pin, symbol SofleKeyboard-rescue:OLED-Lily58-cache-Lily58_Pro-rescue
- removed JP1, JP2, JP3, JP4, JP5, JP6, JP7, JP8: Jumper_NO_Small, SofleChoc:Jumper, symbol SofleKeyboard-rescue:Jumper_NO_Small-Device
- removed P1, P2: i2c_pin, SofleChoc:1pin_conn, symbol SofleKeyboard-rescue:i2c_pin-Lily58-cache-Lily58_Pro-rescue
- removed R1, R2: R, SofleChoc:RESISTOR_mini, symbol SofleKeyboard-rescue:R-Lily58-cache-Lily58_Pro-rescue
- removed RSW1: SW_RST, SofleChoc:TACT_SWITCH_TVBP06, symbol SofleKeyboard-rescue:SW_RST-Lily58-cache-Lily58_Pro-rescue
- removed TH5, TH6, TH7, TH8: HOLE, SofleChoc:M2_HOLE_PCB, symbol SofleKeyboard-rescue:HOLE-Lily58-cache-Lily58_Pro-rescue
- removed TH9: HOLE, SofleChoc:HOLE_M2_TH, symbol SofleKeyboard-rescue:HOLE-Lily58-cache-Lily58_Pro-rescue
- removed W1: jumper, Jumper:SolderJumper-2_P1.3mm_Open_Pad1.0x1.5mm, symbol SofleKeyboard-rescue:Jumper-Device
- added D35, D36, D37, D40, D41, D42, D43: D, SofleChoc:crkbd-diode, symbol SofleKeyboard-rescue:D-Lily58-cache-Lily58_Pro-rescue
- added J_RGB1: RGB jumper, Jumper:SolderJumper-3_P2.0mm_Open_TrianglePad1.0x1.5mm, symbol Jumper:Jumper_3_Open
- added SW35, SW36, SW37, SW38, SW39, SW40, SW41: SW_PUSH_LED, SofleChoc:Choc_Hotswap_SK6812MiniE, symbol SofleKeyboard:SW_PUSH_LED
- U1: value ProMicro -> RP2040; footprint SofleChoc:ProMicro -> RP2040:RP2040-mini
Connections:
- net RESET is gone; now on net DATA: U1.22 (RST)
- net SCL is gone; now on net COL2: U1.6 (SCL(PD0))
- net SDA is gone; now on net COL1: U1.5 (SDA(PD1))
- net i2c_d is gone; now on net DATA: J1.3
- net COL0: now also U1.4 (GND); no longer U1.19 (A2(PF5))
- net COL1: no longer U1.18 (A1(PF6))
- net COL2: no longer U1.17 (A0(PF7))
- net COL3: now also U1.7 (D4(PD4)); no longer U1.16 (D15(PB1))
- net COL4: now also U1.8 (D5(PC6)); no longer U1.15 (D14(PB3))
- net COL5: now also U1.9 (D6(PD7)); no longer U1.14 (D16(PB2))
- net COL6: now also U1.10 (D7(PE6)); no longer U1.13 (D10(PB6))
- net DATA: no longer U1.2 (RX(PD2))
- net GND: now also U1.2 (RX(PD2)), SW35.3 (GND), SW36.3 (GND), SW37.3 (GND), SW38.3 (GND), SW39.3 (GND), SW40.3 (GND), SW41.3 (GND); no longer U1.23 (GND), U1.3 (GND), U1.4 (GND)
- net LED: now also U1.23 (GND), J_RGB1.1 (A), J_RGB1.3 (B); no longer SW1.4 (DIN), U1.1 (TX(PD3))
- net ROW0: now also U1.21 (VCC), D35.1 (K), D40.1 (K); no longer U1.8 (D5(PC6))
- net ROW1: now also U1.20 (A3(PF4)), D36.1 (K), D41.1 (K); no longer U1.9 (D6(PD7))
- net ROW2: now also U1.19 (A2(PF5)), D37.1 (K), D42.1 (K); no longer U1.10 (D7(PE6))
- net ROW3: now also U1.18 (A1(PF6)), D43.1 (K); no longer U1.11 (D8(PB4))
- net ROW4: now also U1.17 (A0(PF7)); no longer U1.12 (D9(PB5))
- net VCC: now also U1.3 (GND), SW35.1 (VDD), SW36.1 (VDD), SW37.1 (VDD), SW38.1 (VDD), SW39.1 (VDD), SW40.1 (VDD), SW41.1 (VDD); no longer U1.21 (VCC)
- net at SW8.2 (DOUT): now also SW36.4 (DIN); no longer SW15.4 (DIN)
- net at SW15.2 (DOUT): now also SW38.4 (DIN); no longer SW22.4 (DIN)
- net i2c_c renamed led_bridge
- new net: SW1.4 (DIN), SW35.2 (DOUT)
- new net: SW15.4 (DIN), SW37.2 (DOUT)
- new net: SW22.4 (DIN), SW38.2 (DOUT)
- new net: SW37.4 (DIN), SW39.2 (DOUT)
- new net: SW39.4 (DIN), SW40.2 (DOUT)
- new net: D40.2 (A), SW35.5
- new net: D43.2 (A), SW38.5
- new net: D41.2 (A), SW36.5
- new net: SW36.2 (DOUT), SW40.4 (DIN)
- new net: D37.2 (A), SW39.5
- new net: D35.2 (A), SW41.5
- new net: SW35.4 (DIN), SW41.2 (DOUT)
- new net: D36.2 (A), SW40.5
- new net: D42.2 (A), SW37.5
- new net COL7: SW35.6, SW36.6, SW37.6, SW38.6, U1.11 (D8(PB4))
- new net COL8: SW39.6, SW40.6, SW41.6, U1.12 (D9(PB5))
- new net LED_start: J_RGB1.2 (C), SW41.4 (DIN)
- no-connect marks 4 -> 6
