File: PCB/NomadKeyboard.kicad_sch (KiCad schematic)
At the start: 89 parts, among them J1 4PIN, SW1 SW_PUSH_LED, SW10 SW_PUSH_LED, SW11 SW_PUSH_LED, SW12 SW_PUSH_LED, SW13 SW_PUSH_LED, SW14 SW_PUSH_LED, SW15 SW_PUSH_LED, SW16 SW_PUSH_LED, SW17 SW_PUSH_LED, SW18 SW_PUSH_LED, SW19 SW_PUSH_LED, SW2 SW_PUSH_LED, SW20 SW_PUSH_LED, SW21 SW_PUSH_LED, SW22 SW_PUSH_LED, SW23 SW_PUSH_LED, SW24 SW_PUSH_LED, SW25 SW_PUSH_LED, SW26 SW_PUSH_LED, SW27 SW_PUSH_LED, SW28 SW_PUSH_LED, SW29 SW_PUSH_LED, SW3 SW_PUSH_LED, SW30 SW_PUSH_LED, SW31 SW_PUSH_LED, SW32 SW_PUSH_LED, SW33 SW_PUSH_LED, SW34 SW_PUSH_LED, SW35 SW_PUSH_LED, SW36 SW_PUSH_LED, SW37 SW_PUSH_LED, SW38 SW_PUSH_LED, SW39 SW_PUSH_LED, SW4 SW_PUSH_LED, SW40 SW_PUSH_LED, SW41 SW_PUSH_LED, SW5 SW_PUSH_LED, SW6 SW_PUSH_LED, SW7 SW_PUSH_LED, SW8 SW_PUSH_LED, SW9 SW_PUSH_LED, U1 RP2040

Commit message: Finished, updated gerber files
Parts:
- added SW42: RotaryEncoder_Switch, Rotary_Encoder:RotaryEncoder_Alps_EC11E-Switch_Vertical_H20mm, symbol Device:RotaryEncoder_Switch
Connections:
- net GND: now also SW42.C, SW42.S2
- net LED: no longer J_RGB1.3 (B)
- net led_bridge: now also SW34.2 (DOUT)
- net enc_i: now reaches U1.13 (D10(PB6))
- net enc_i: now also SW42.B
- net enc_d: now reaches U1.14 (D16(PB2))
- net enc_d: now also SW42.A
- net enc_s: now reaches U1.16 (D15(PB1))
- net enc_s: now also SW42.S1
- new net LED_slave: J_RGB1.3 (B)
- no-connect marks 6 -> 2
